File: hw-output/20-000-Schema Elettrico/10000002.sch (KiCad schematic (older format))
At the start: 26 parts, among them P1 CONN_4, P2 CONN_4, P3 CONN_4, P4 CONN_4, P5 CONN_4, P6 CONN_4, P7 CONN_4, P8 CONN_4, U1 PCF8574, U2 AQZ204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

Commit message: Aggiunte capacità di bypass su alimentazione I2C expander
Parts:
- added C1: 100n, Capacitors_SMD:C_0603_HandSoldering, symbol C
- added C2: 1u, Capacitors_SMD:C_0603_HandSoldering, symbol C
- R1, R10, R11, R12, R13, R2, R3, R4, R5, R6, R7, R8, R9: footprint ~ -> (none)
- U2, U3: footprint MODULE -> (none)
Connections:
- wire segments 105 -> 111

Commit message: Inizio nuovo schema versione 02
Parts:
- removed C1: 100n, Capacitors_SMD:C_0603_HandSoldering, symbol C
- removed C2: 1u, Capacitors_SMD:C_0603_HandSoldering, symbol C
- removed D1, D2: ZENERSMALL, symbol ZENERSMALL
- removed P1, P2, P3, P4, P5, P6, P7, P8: CONN_4, symbol CONN_4
- removed R1, R2, R3, R4, R5, R6: 0, symbol R
- removed R10, R12: 1000, symbol R
- removed R11, R13, R7, R8, R9: 10000, symbol R
- removed U1: PCF8574, symbol PCF8574
- added C?: C_100n_0603_10_X7R_25V, Capacitors_SMD:C_0603, symbol C_100n_0603_10_X7R_25V
- added C?: C_1u_0603_10_X7R_25V, Capacitors_SMD:C_0603, symbol C_1u_0603_10_X7R_25V
- added D? (x2): TVS_SMC_49.1V, Diodes_SMD:SMC_Standard, symbol TVS_SMC_49.1V
- added P? (x8): PLUG_01X04_254, Socket_Strips:Socket_Strip_Straight_1x04, symbol PLUG_01X04_254
- added R? (x6): R_0_0603_5, Resistors_SMD:R_0603, symbol R_0_0603_5
- added R? (x3): R_10K_0603_5, Resistors_SMD:R_0603, symbol R_10K_0603_5
- added U?: TCA9554, Housings_SSOP:SSOP-16_3.9x4.9mm_Pitch0.635mm, symbol TCA9554
Connections:
- net labels added: +5V
- wire segments 111 -> 109

Commit message: Terminato schema uscite
Parts:
- removed U2, U3: AQZ204, symbol AQZ204
- added Q? (x2): Q_PMOS_GSD_BSS84, TO_SOT_Packages_SMD:SOT-23, symbol Q_PMOS_GSD_BSS84
- added R? (x4): R_1K_0603_5, Resistors_SMD:R_0603, symbol R_1K_0603_5
- added R? (x4): R_10K_0603_5, Resistors_SMD:R_0603, symbol R_10K_0603_5
- added U? (x2): AQZ204, os_photomos:AQZ-SIL-4, symbol AQZ204
Connections:
- net labels removed: VDD
- wire segments 109 -> 119
Other:
- moved on the sheet: D?, P?

Commit message: Completato schema e sbroglio
Signed-off-by: CrazyDiamond <crazyd14@gmail.com>
Parts:
- removed P? (x2): PLUG_01X04_254, Socket_Strips:Socket_Strip_Straight_1x04, symbol PLUG_01X04_254
- added P1, P2: TERMINAL_01X04_250_RA_SPRING, os_terminal_block:1770908, symbol TERMINAL_01X04_250_RA_SPRING
- gave numbers to parts that had none: 32
