File: hw-temp/20-000-Schema Elettrico/10000006_SE.kicad_pcb (KiCad board)
At the start: 4 copper layers, 45.8 x 32.3 mm, 39 parts, among them P1 PLUG_01X04_254, P2 PLUG_01X04_254, P3 PLUG_01X04_254, P4 PLUG_01X04_254, P5 PLUG_01X04_254, P6 PLUG_01X04_254, P7 PLUG_01X04_254, P8 PLUG_01X04_254, U1 TPS709, U2 PCA9306DC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

Commit message: Pulizia schema
Parts:
- moved R11 10.9 mm to (183.4, 128.7)
- moved R10 10.2 mm to (178.1, 131.7), turned to 0 degrees
- moved R9 9.65 mm to (178.1, 130.0), turned to 0 degrees
- moved R8 8.30 mm to (173.7, 138.4), turned to 180 degrees
- moved R7 6.83 mm to (183.0, 138.7)
- moved R3 5.83 mm to (188.6, 143.6), turned to 0 degrees
- moved R4 5.83 mm to (188.6, 142.0), turned to 180 degrees
- moved R1 3.30 mm to (183.0, 142.0)
- moved R2 3.30 mm to (183.0, 143.6)
- moved C6 2.03 mm to (177.5, 142.2)
- moved C3 2.03 mm to (173.7, 142.2)
- moved C4 2.03 mm to (173.7, 140.7)
- moved C5 2.03 mm to (177.5, 140.7)
- moved R5 1.88 mm to (188.6, 138.7)
- moved R6 1.88 mm to (188.6, 140.3)
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Routing:
- net /I2C_SCL: track 0.00 -> 48.5 mm
- net /I2C_SDA: track 0.00 -> 44.4 mm
- net GND: track 0.00 -> 40.5 mm, vias 0 -> 14
- net +3V3: track 0.00 -> 39.4 mm, vias 0 -> 13
- net /GPIO0: track 0.00 -> 32.7 mm, vias 0 -> 2
- net /DATA_RDYn: track 0.00 -> 30.4 mm, vias 0 -> 2
- net /RTDIN_N: track 0.00 -> 22.8 mm, vias 0 -> 1
- net /SPI_MISO: track 0.00 -> 20.0 mm, vias 0 -> 2
- net +5V: track 0.00 -> 18.7 mm, vias 0 -> 1
- net /FORCE_N: track 0.00 -> 18.0 mm, vias 0 -> 1
- net /SPI_MOSI: track 0.00 -> 16.4 mm, vias 0 -> 2
- net /FORCE_P: track 0.00 -> 16.2 mm, vias 0 -> 1
- net Net-(R1-Pad1): track 0.00 -> 15.8 mm
- net /I2C_SCL_3V3: track 0.00 -> 15.4 mm
- net /RTDIN_P: track 0.00 -> 14.5 mm, vias 0 -> 2
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- added copper zone on In1.Cu, net +3V3
- added copper zone on In1.Cu, net +5V
- removed copper zone on F.Cu, net +3V3
- removed copper zone on F.Cu, net +5V

Commit message: completato schema elettrico e sbroglio
Signed-off-by: CrazyDiamond <crazyd14@gmail.com>
Parts:
- added R17: R_0_0603_5, Resistors_SMD:R_0603, F.Cu at (173.1, 131.7)
Routing:
- net +5V: track 18.7 -> 22.0 mm
- net +3V3: track 39.4 -> 40.8 mm, vias 13 -> 14
Changed lines of the file:
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@@
 (kicad_pcb (version 4) (host pcbnew 4.0.1-stable)
   (general
-    (links 84)
-    (no_connects 67)
+    (links 86)
+    (no_connects 2)
     (area 166.421999 119.304999 212.419001 151.713001)
     (thickness 1.6)
     (drawings 96)
-    (tracks 333)
+    (tracks 341)
     (zones 0)
-    (modules 39)
+    (modules 40)
     (nets 48)
   )
@@
     (tags "resistor 0603")
     (attr smd)
-    (fp_text reference R10 (at -3.175 0) (layer F.SilkS)
+    (fp_text reference R10 (at 2.667 0) (layer F.SilkS)
       (effects (font (size 1 1) (thickness 0.15)))
     )
@@
     (tags SOT-23-5)
     (attr smd)
-    (fp_text reference U1 (at -1.313 2.667) (layer F.SilkS)
+    (fp_text reference U1 (at -0.424 -2.54) (layer F.SilkS)
       (effects (font (size 1 1) (thickness 0.15)))
     )
@@
     (pad 2 smd rect (at 0.75 0 180) (size 0.5 0.9) (layers F.Cu F.Paste F.Mask)
       (net 35 /GPIO0))
+    (model Resistors_SMD.3dshapes/R_0603.wrl
+      (at (xyz 0 0 0))
+      (scale (xyz 1 1 1))
+      (rotate (xyz 0 0 0))
+    )
+  )
+  (module Resistors_SMD:R_0603 (layer F.Cu)
+    (at 173.101 131.699 180)
+    (descr "Resistor SMD 0603, reflow soldering, Vishay (see dcrcw.pdf)")
+    (tags "resistor 0603")
+    (attr smd)
+    (fp_text reference R17 (at 0.762 1.651 180) (layer F.SilkS)
+      (effects (font (size 1 1) (thickness 0.15)))
+    )
+    (fp_text value R_0_0603_5 (at 0 1.9 180) (layer F.Fab)
+      (effects (font (size 1 1) (thickness 0.15)))
+    )
+    (fp_line (start -1.3 -0.8) (end 1.3 -0.8) (layer F.CrtYd) (width 0.05))
+    (fp_line (start -1.3 0.8) (end 1.3 0.8) (layer F.CrtYd) (width 0.05))
+    (fp_line (start -1.3 -0.8) (end -1.3 0.8) (layer F.CrtYd) (width 0.05))
+    (fp_line (start 1.3 -0.8) (end 1.3 0.8) (layer F.CrtYd) (width 0.05))
+    (fp_line (start 0.5 0.675) (end -0.5 0.675) (layer F.SilkS) (width 0.15))
+    (fp_line (start -0.5 -0.675) (end 0.5 -0.675) (layer F.SilkS) (width 0.15))
+    (pad 1 smd rect (at -0.75 0 180) (size 0.5 0.9) (layers F.Cu F.Paste F.Mask)
+      (net 3 +3V3))
+    (pad 2 smd rect (at 0.75 0 180) (size 0.5 0.9) (layers F.Cu F.Paste F.Mask)
+      (net 1 +5V))
     (model Resistors_SMD.3dshapes/R_0603.wrl
       (at (xyz 0 0 0))
@@
   (gr_line (start 166.5605 151.4996) (end 212.2805 151.4996) (layer Dwgs.User) (width 0.1))
   (gr_line (start 166.5605 151.5986) (end 212.2805 151.5986) (layer Dwgs.User) (width 0.1))
+  (segment (start 172.351 131.699) (end 171.851 131.699) (width 0.25) (layer F.Cu) (net 1))
+  (segment (start 171.851 131.699) (end 169.037 131.699) (width 0.25) (layer F.Cu) (net 1))
   (segment (start 173.237 135.453) (end 172.437 135.453) (width 0.25) (layer F.Cu) (net 1))
   (segment (start 172.437 135.453) (end 171.958 135.932) (width 0.25) (layer F.Cu) (net 1))
@@
   (segment (start 172.552 127.381) (end 171.772 127.381) (width 0.25) (layer F.Cu) (net 2))
   (segment (start 171.772 127.381) (end 171.391 127.762) (width 0.25) (layer F.Cu) (net 2))
+  (via (at 174.879 131.699) (size 0.6) (drill 0.4) (layers F.Cu B.Cu) (net 3))
+  (segment (start 174.093 131.699) (end 174.879 131.699) (width 0.25) (layer F.Cu) (net 3))
+  (segment (start 173.851 131.457) (end 174.093 131.699) (width 0.25) (layer F.Cu) (net 3))
+  (segment (start 173.851 131.699) (end 173.851 131.457) (width 0.25) (layer F.Cu) (net 3))
   (via (at 191.008 134.112) (size 0.6) (drill 0.4) (layers F.Cu B.Cu) (net 3))
   (segment (start 190.556 134.564) (end 191.008 134.112) (width 0.25) (layer F.Cu) (net 3))
@@
   (segment (start 195.961 129.032) (end 195.199 129.794) (width 0.25) (layer F.Cu) (net 5))
   (segment (start 195.199 129.794) (end 195.199 133.589) (width 0.25) (layer F.Cu) (net 5))
+  (segment (start 169.037 134.239) (end 170.815 134.239) (width 0.25) (layer F.Cu) (net 6))
+  (segment (start 174.625 134.549) (end 174.371 134.803) (width 0.25) (layer F.Cu) (net 6))
+  (segment (start 170.815 134.239) (end 172.212 132.842) (width 0.25) (layer F.Cu) (net 6))
+  (segment (start 172.212 132.842) (end 174.371 132.842) (width 0.25) (layer F.Cu) (net 6))
+  (segment (start 174.371 132.842) (end 174.625 133.096) (width 0.25) (layer F.Cu) (net 6))
+  (segment (start 174.371 134.803) (end 173.237 134.803) (width 0.25) (layer F.Cu) (net 6))
+  (segment (start 174.625 133.096) (end 174.625 134.549) (width 0.25) (layer F.Cu) (net 6))
   (segment (start 174.117 122.301) (end 174.117 123.567) (width 0.25) (layer In2.Cu) (net 6))
   (segment (start 174.117 123.567) (end 172.716 124.968) (width 0.25) (layer In2.Cu) (net 6))
@@
   (segment (start 167.005 127.254) (end 167.005 133.477) (width 0.25) (layer In2.Cu) (net 6))
   (segment (start 167.005 133.477) (end 167.767 134.239) (width 0.25) (layer In2.Cu) (net 6))
-  (segment (start 173.237 134.803) (end 174.442 134.803) (width 0.25) (layer F.Cu) (net 6))
-  (segment (start 174.442 134.803) (end 174.879 134.366) (width 0.25) (layer F.Cu) (net 6))
-  (segment (start 174.879 134.366) (end 174.879 133.35) (width 0.25) (layer F.Cu) (net 6))
-  (segment (start 174.879 133.35) (end 174.371 132.842) (width 0.25) (layer F.Cu) (net 6))
-  (segment (start 174.371 132.842) (end 172.212 132.842) (width 0.25) (layer F.Cu) (net 6))
-  (segment (start 172.212 132.842) (end 170.815 134.239) (width 0.25) (layer F.Cu) (net 6))
-  (segment (start 170.815 134.239) (end 169.037 134.239) (width 0.25) (layer F.Cu) (net 6))
   (segment (start 174.117 148.971) (end 174.117 147.705) (width 0.25) (layer In2.Cu) (net 6))
   (segment (start 174.117 147.705) (end 173.228 146.816) (width 0.25) (layer In2.Cu) (net 6))
@@
   (segment (start 174.486 137.002) (end 173.587 136.103) (width 0.25) (layer F.Cu) (net 30))
   (segment (start 173.587 136.103) (end 173.237 136.103) (width 0.25) (layer F.Cu) (net 30))
+  (segment (start 177.537 135.453) (end 176.093 135.453) (width 0.25) (layer F.Cu) (net 31))
+  (segment (start 176.093 135.453) (end 175.768 135.128) (width 0.25) (layer F.Cu) (net 31))
+  (segment (start 175.768 135.128) (end 175.768 131.75699) (width 0.25) (layer F.Cu) (net 31))
+  (segment (start 175.768 131.75699) (end 175.95299 131.572) (width 0.25) (layer F.Cu) (net 31))
+  (segment (start 175.95299 130.37101) (end 176.276 130.048) (width 0.25) (layer F.Cu) (net 31))
+  (segment (start 175.95299 131.572) (end 175.95299 130.37101) (width 0.25) (layer F.Cu) (net 31))
+  (segment (start 176.276 130.048) (end 177.304 130.048) (width 0.25) (layer F.Cu) (net 31))
   (segment (start 177.537 135.453) (end 177.593 135.509) (width 0.25) (layer F.Cu) (net 31))
   (segment (start 177.593 135.509) (end 178.278002 135.509) (width 0.25) (layer F.Cu) (net 31))
@@
   (segment (start 178.943 136.779) (end 179.451 137.287) (width 0.25) (layer F.Cu) (net 31))
   (segment (start 179.451 137.287) (end 182.361 137.287) (width 0.25) (layer F.Cu) (net 31))
-  (segment (start 177.537 135.453) (end 176.093 135.453) (width 0.25) (layer F.Cu) (net 31))
-  (segment (start 176.093 135.453) (end 175.641 135.001) (width 0.25) (layer F.Cu) (net 31))
-  (segment (start 175.641 130.683) (end 176.276 130.048) (width 0.25) (layer F.Cu) (net 31))
-  (segment (start 175.641 135.001) (end 175.641 130.683) (width 0.25) (layer F.Cu) (net 31))
-  (segment (start 176.276 130.048) (end 177.304 130.048) (width 0.25) (layer F.Cu) (net 31))
+  (segment (start 176.657 131.699) (end 176.403 131.953) (width 0.25) (layer F.Cu) (net 32))
+  (segment (start 176.403 134.493) (end 176.403 131.953) (width 0.25) (layer F.Cu) (net 32))
+  (segment (start 176.657 134.747) (end 176.926 134.747) (width 0.25) (layer F.Cu) (net 32))
+  (segment (start 176.657 134.747) (end 176.403 134.493) (width 0.25) (layer F.Cu) (net 32))
+  (segment (start 177.304 131.699) (end 176.657 131.699) (width 0.25) (layer F.Cu) (net 32))
+  (segment (start 176.982 134.803) (end 177.537 134.803) (width 0.25) (layer F.Cu) (net 32))
+  (segment (start 176.926 134.747) (end 176.982 134.803) (width 0.25) (layer F.Cu) (net 32))
   (segment (start 183.134 135.864) (end 183.034001 135.963999) (width 0.25) (layer F.Cu) (net 32))
   (segment (start 183.034001 135.963999) (end 181.790001 135.963999) (width 0.25) (layer F.Cu) (net 32))
@@
   (segment (start 180.213 136.525) (end 178.491 134.803) (width 0.25) (layer F.Cu) (net 32))
   (segment (start 178.491 134.803) (end 177.537 134.803) (width 0.25) (layer F.Cu) (net 32))
-  (segment (start 176.09101 132.26499) (end 176.657 131.699) (width 0.25) (layer F.Cu) (net 32))
-  (segment (start 176.657 131.699) (end 177.304 131.699) (width 0.25) (layer F.Cu) (net 32))
-  (segment (start 176.09101 134.56201) (end 176.09101 132.26499) (width 0.25) (layer F.Cu) (net 32))
-  (segment (start 176.926 134.747) (end 176.276 134.747) (width 0.25) (layer F.Cu) (net 32))
-  (segment (start 176.276 134.747) (end 176.09101 134.56201) (width 0.25) (layer F.Cu) (net 32))
-  (segment (start 177.537 134.803) (end 176.982 134.803) (width 0.25) (layer F.Cu) (net 32))
-  (segment (start 176.982 134.803) (end 176.926 134.747) (width 0.25) (layer F.Cu) (net 32))
   (segment (start 182.638 128.651) (end 181.61 128.651) (width 0.25) (layer F.Cu) (net 33))
   (segment (start 181.61 128.651) (end 181.229 129.032) (width 0.25) (layer F.Cu) (net 33))

Commit message: PCB terminato
Signed-off-by: CrazyDiamond <crazyd14@gmail.com>
Parts:
- P1, P2: value PLUG_01X04_254 -> TERMINAL_01X04_250_RA_SPRING; footprint Socket_Strips:Socket_Strip_Straight_1x04 -> os_terminal_block:1770908
- R1, R13, R14, R15, R2, R3, R4, R5, R6, R7: moved to B.Cu
- moved R2 15.4 mm to (184.1, 128.2)
- moved R6 14.0 mm to (190.1, 126.5)
- moved R3 13.9 mm to (190.1, 129.9)
- moved R7 12.2 mm to (184.1, 126.5)
- moved R1 12.2 mm to (184.1, 129.9)
- moved R11 12.0 mm to (195.2, 126.4)
- moved R5 10.7 mm to (190.1, 128.1)
- moved R4 10.6 mm to (190.1, 131.5)
- moved R15 8.76 mm to (199.1, 137.1)
- moved R13 8.42 mm to (199.1, 138.9), turned to 180 degrees
- moved C3 6.80 mm to (179.8, 145.2)
- moved C4 6.80 mm to (179.8, 143.7)
- moved R8 6.80 mm to (179.8, 141.4)
- moved C5 6.80 mm to (183.6, 143.7)
- moved C6 6.80 mm to (183.6, 145.2)
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Connections:
- P4 pad 1: Net-(P4-Pad1) -> (no net)
- P4 pad 2: Net-(P4-Pad2) -> (no net)
- P4 pad 3: Net-(P4-Pad3) -> (no net)
- P4 pad 4: Net-(P4-Pad4) -> (no net)
- P5 pad 1: Net-(P5-Pad1) -> (no net)
- P5 pad 2: Net-(P5-Pad2) -> (no net)
- P5 pad 3: Net-(P5-Pad3) -> (no net)
- P5 pad 4: Net-(P5-Pad4) -> (no net)
- P7 pad 1: Net-(P7-Pad1) -> (no net)
- P7 pad 2: Net-(P7-Pad2) -> (no net)
- P7 pad 3: Net-(P7-Pad3) -> (no net)
- P7 pad 4: Net-(P7-Pad4) -> (no net)
- P8 pad 1: Net-(P8-Pad1) -> (no net)
- P8 pad 2: Net-(P8-Pad2) -> (no net)
- P8 pad 3: Net-(P8-Pad3) -> (no net)
- P8 pad 4: Net-(P8-Pad4) -> (no net)
- U1 pad 3: Net-(U1-Pad3) -> (no net)
- U1 pad 4: Net-(U1-Pad4) -> (no net)
- U3 pad 10: /GPIO2 -> (no net)
- U3 pad 13: /GPIO3 -> (no net)
- U3 pad 9: /INT0n -> (no net)
- U4 pad 20: Net-(U4-Pad20) -> (no net)
Routing:
- net /DATA_RDYn: track 30.4 -> 16.8 mm
- net +5V: track 22.0 -> 30.0 mm, vias 1 -> 2
- net Net-(R1-Pad1): track 15.8 -> 7.84 mm, vias 0 -> 1
- net /SPI_CLK: track 6.57 -> 14.2 mm
- net Net-(R3-Pad1): track 14.4 -> 7.69 mm, vias 0 -> 1
- net /BIAS: track 12.1 -> 5.46 mm, vias 0 -> 1
- net /FORCE_N: track 18.0 -> 24.6 mm, vias 1 -> 0
- net /I2C_SCL: track 48.3 -> 54.5 mm
- net /I2C_SDA: track 44.4 -> 50.2 mm
- net /GPIO1: track 6.82 -> 12.5 mm
- net /ISENSOR: track 9.93 -> 5.90 mm, vias 0 -> 1
- net /FORCE_P: track 16.2 -> 12.8 mm
- net /FORCE2: track 7.83 -> 4.68 mm, vias 0 -> 1
- net Net-(R5-Pad1): track 8.15 -> 5.03 mm, vias 0 -> 1
- net /GPIO0: track 32.7 -> 29.7 mm
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Other:
- rule trace_min: 0.2 -> 0.1
